Commit message: new urdf and finger follower

File: test_ws/src/jessica_description/description/dimensions.xacro (robot description, xacro)
@@ -46,6 +46,15 @@
   <xacro:property name="servo_width"  value="0.0197"/>
   <xacro:property name="servo_height" value="0.0429"/>
-  <!-- Standoff from the pan servo's output shaft to the tilt servo's output
-       shaft ("tilt attachment around 5cm tall"). -->
-  <xacro:property name="tilt_bracket_height" value="0.05"/>
+  <!-- Coupler between the pan servo's output and the tilt servo. -->
+  <xacro:property name="pan_tilt_spacer_height" value="0.01"/>
+  <!-- U-bracket the head sits on, straddling the tilt servo's rotation axis. -->
+  <xacro:property name="head_bracket_height"       value="0.05"/>
+  <xacro:property name="head_bracket_arm_spacing"   value="0.03"/>
+  <xacro:property name="head_bracket_arm_thickness" value="0.006"/>
+  <!-- Stereo camera on the head. camera_face_x/z are the head's front
+       surface and vertical mid-height (head_bottom+head_top combined bounding
+       box), relative to the head link's own origin - see stereo_camera.xacro. -->
+  <xacro:property name="camera_baseline" value="0.062"/>
+  <xacro:property name="camera_face_x"   value="0.051776"/>
+  <xacro:property name="camera_face_z"   value="0.113845"/>
 </robot>

File: test_ws/src/jessica_description/description/frame.xacro (robot description, xacro)
@@ -31,5 +31,5 @@
 -->
 <robot xmlns:xacro="http://www.ros.org/wiki/xacro">
-  <xacro:macro name="frame_mesh_part" params="mesh_name xyz rpy box_size">
+  <xacro:macro name="frame_mesh_part" params="mesh_name xyz rpy box_size material:=gray">
     <visual>
       <origin xyz="${xyz}" rpy="${rpy}"/>
@@ -37,5 +37,5 @@
         <mesh filename="package://jessica_description/description/meshes/visual/${mesh_name}.stl" scale="0.001 0.001 0.001"/>
       </geometry>
-      <material name="gray"/>
+      <material name="${material}"/>
     </visual>
     <collision>
@@ -88,4 +88,24 @@
     <xacro:frame_mesh_part mesh_name="body_432" box_size="${channel_cross} ${body_length} ${channel_cross}"
       xyz="${body_x} ${-foot_track_y - 0.0215} ${grid_top_z}" rpy="${pi/2} 0 0"/>
+    <!-- Front panel (wife_boobs_v2_13.stl) - a bowl shape; flat rim (the
+         mesh's flat reference plane) goes against the body, curved bottom
+         sticks out forward. rpy=(90,90,-90)deg (URDF fixed-axis roll/pitch/yaw)
+         puts the rotated bounding box at X in [0, 66.993], Y in [-76.9997,
+         66.9998], Z in [-52, 68.951] before translation - the rim lands
+         exactly at rotated X=0 with no correction needed, which is a good
+         sign this orientation (vs. the previous +90deg yaw) is the right one:
+           - top-aligned: rotated Z-max (68.951mm) placed at body_top_z
+           - right-aligned: rotated Y-min (-76.9997mm) placed at the right
+             body channel's outer face
+           - forward-touching: rotated X-min (0, the rim) placed at the
+             body's front face, bowl curving forward from there -->
+    <xacro:frame_mesh_part mesh_name="robot_front" material="white" box_size="0.121 0.144 0.067"
+      xyz="${body_x + channel_cross/2} ${-(foot_track_y + channel_cross/2) + 0.077000} ${body_top_z - 0.068951}" rpy="${pi/2} ${pi/2} ${-pi/2}"/>
+    <!-- Same part, mirrored to the left side. The rotated bounding box isn't
+         symmetric in Y (-76.9997 to 66.9998), so this isn't just the negative
+         of the right copy's Y - it's the *other* extreme (rotated Y-max)
+         placed at the left body channel's outer face. -->
+    <xacro:frame_mesh_part mesh_name="robot_front" material="white" box_size="0.121 0.144 0.067"
+      xyz="${body_x + channel_cross/2} ${foot_track_y + channel_cross/2 - 0.067000} ${body_top_z - 0.068951}" rpy="${pi/2} ${pi/2} ${-pi/2}"/>
   </link>
   <joint name="body_top_joint" type="fixed">

File: test_ws/src/jessica_description/description/jessica.urdf.xacro (robot description, xacro)
@@ -18,4 +18,5 @@
   <xacro:include filename="wheels.xacro"/>
   <xacro:include filename="pan_tilt.xacro"/>
+  <xacro:include filename="stereo_camera.xacro"/>
   <xacro:if value="$(arg use_ros2_control)">
     <xacro:include filename="ros2_control.xacro"/>

File: test_ws/src/jessica_description/description/pan_tilt.xacro (robot description, xacro)
@@ -2,6 +2,6 @@
 <!--
   Pan-tilt head assembly: two MG996-form-factor servos, pan on the bottom,
-  tilt on top of a ~50mm standoff bracket, real head mesh
-  (eva_head_frontBottom-part.stl) mounted on the tilt output.
+  tilt on top of a ~10mm coupler, real head mesh mounted on a 50mm U-bracket
+  on the tilt output.
   This replaces the old placeholder "mast" - the pan servo now sits on a
   short 5mm neck riser on top of `body_top` (see frame.xacro), so the head
@@ -28,5 +28,5 @@
     <parent link="body_top"/>
     <child  link="neck"/>
-    <origin xyz="0 0 0" rpy="0 0 0"/>
+    <origin xyz="0.005 0 0" rpy="0 0 0"/>
   </joint>
   <link name="neck">
@@ -59,15 +59,19 @@
   </joint>
   <link name="tilt_mount">
+    <!-- coupler between the pan servo's output and the tilt servo -->
     <visual>
-      <origin xyz="0 0 ${tilt_bracket_height/2}" rpy="0 0 0"/>
-      <geometry><box size="0.02 0.02 ${tilt_bracket_height}"/></geometry>
+      <origin xyz="0 0 ${pan_tilt_spacer_height/2}" rpy="0 0 0"/>
+      <geometry><cylinder radius="0.008" length="${pan_tilt_spacer_height}"/></geometry>
       <material name="gray"/>
     </visual>
     <collision>
-      <origin xyz="0 0 ${tilt_bracket_height/2}" rpy="0 0 0"/>
-      <geometry><box size="0.02 0.02 ${tilt_bracket_height}"/></geometry>
+      <origin xyz="0 0 ${pan_tilt_spacer_height/2}" rpy="0 0 0"/>
+      <geometry><cylinder radius="0.008" length="${pan_tilt_spacer_height}"/></geometry>
     </collision>
-    <!-- tilt servo mounted at the top of the bracket, shaft (servo_height axis) horizontal along Y -->
-    <xacro:mg996_servo xyz="0 0 ${tilt_bracket_height}" rpy="${pi/2} 0 0"/>
+    <!-- tilt servo mounted directly on top of the coupler, shaft (servo_height axis) horizontal along Y.
+         Box origin = box centre, so its bottom edge (half of servo_width,
+         the rotated box's vertical extent) needs to sit at the coupler's
+         top - otherwise the box swallows most of the cylinder below it. -->
+    <xacro:mg996_servo xyz="0 0 ${pan_tilt_spacer_height + servo_width/2}" rpy="${pi/2} 0 0"/>
   </link>
   <!-- tilt: pitch about Y -->
@@ -75,12 +79,45 @@
     <parent link="tilt_mount"/>
     <child  link="head"/>
-    <origin xyz="0 0 ${tilt_bracket_height}" rpy="0 0 0"/>
+    <origin xyz="0 0 ${pan_tilt_spacer_height + servo_width/2}" rpy="0 0 0"/>
     <axis xyz="0 1 0"/>
     <limit lower="-1.5" upper="0.87" effort="5.0" velocity="3.0"/>
   </joint>
   <link name="head">
+    <!-- U-bracket the head sits on, straddling the tilt servo's rotation
+         axis (Y) with an arm on each side, rising to head_bracket_height. -->
     <visual>
-      <origin xyz="0 0 0" rpy="0 0 0"/>
+      <origin xyz="0 ${head_bracket_arm_spacing/2} ${head_bracket_height/2}" rpy="0 0 0"/>
+      <geometry><box size="0.03 ${head_bracket_arm_thickness} ${head_bracket_height}"/></geometry>
+      <material name="gray"/>
+    </visual>
+    <collision>
+      <origin xyz="0 ${head_bracket_arm_spacing/2} ${head_bracket_height/2}" rpy="0 0 0"/>
+      <geometry><box size="0.03 ${head_bracket_arm_thickness} ${head_bracket_height}"/></geometry>
+    </collision>
+    <visual>
+      <origin xyz="0 ${-head_bracket_arm_spacing/2} ${head_bracket_height/2}" rpy="0 0 0"/>
+      <geometry><box size="0.03 ${head_bracket_arm_thickness} ${head_bracket_height}"/></geometry>
+      <material name="gray"/>
+    </visual>
+    <collision>
+      <origin xyz="0 ${-head_bracket_arm_spacing/2} ${head_bracket_height/2}" rpy="0 0 0"/>
+      <geometry><box size="0.03 ${head_bracket_arm_thickness} ${head_bracket_height}"/></geometry>
+    </collision>
+    <!-- head mesh sits on top of the bracket. head_bottom.stl's own bottom
+         surface is 43.758mm below its mesh origin (bounding-box zmin), so
+         the origin needs to sit that much above head_bracket_height for the
+         head's actual bottom face - not its origin point - to land on the
+         bracket top. -->
+    <visual>
+      <origin xyz="0.04 0 ${head_bracket_height + 0.043758}" rpy="0 0 0"/>
       <geometry><mesh filename="package://jessica_description/description/meshes/visual/head_bottom.stl" scale="0.001 0.001 0.001"/></geometry>
+      <material name="white"/>
+    </visual>
+    <!-- head_top's bounding box lines up with head_bottom's almost exactly
+         (same Y symmetry, same X range) - both STLs share a common native
+         origin from the same assembly, so the same offset applies here too. -->
+    <visual>
+      <origin xyz="0.04 0 ${head_bracket_height + 0.043758}" rpy="0 0 0"/>
+      <geometry><mesh filename="package://jessica_description/description/meshes/visual/head_top.stl" scale="0.001 0.001 0.001"/></geometry>
       <material name="white"/>
     </visual>
