Commit message: a few fixes

File: from_pi/src/jessica_description/description/dimensions.xacro (robot description, xacro)
@@ -21,5 +21,5 @@
        flag any of these that don't match the real build). -->
   <xacro:property name="wheel_end_inset" value="0.024"/>  <!-- wheel axle inset from each end of a foot -->
-  <xacro:property name="wheel_side_gap"  value="0.020"/>  <!-- gap from the foot's outer face to the wheel's near edge -->
+  <xacro:property name="wheel_side_gap"  value="0.005"/>  <!-- gap from the foot's outer face to the wheel's near edge -->
   <xacro:property name="leg_from_back"   value="0.072"/>  <!-- leg centerline, measured from the back of the foot -->
   <xacro:property name="cross_bar_from_front" value="0.144"/>  <!-- cross-bar centerline, measured from the front of the feet -->

File: from_pi/src/jessica_description/description/ros2_control.xacro (robot description, xacro)
@@ -7,5 +7,5 @@
       <param name="baud_rate">115200</param>
       <param name="timeout_ms">25</param>   <!-- MUST be < loop period (33ms@30Hz). ReadLine blocks the RT loop up to this long when the ESP32 doesn't reply. -->
-      <param name="wheel_radius">7.2</param>        <!-- cm, used by hardware protocol -->
+      <param name="wheel_radius">6.0</param>        <!-- cm, used by hardware protocol (gobilda 3601-0014-0120; scales wheel speed + encoder odom) -->
       <param name="enc_counts_per_rev">1425</param>
     </hardware>

Commit message: lots of changes

File: from_pi/src/jessica_description/description/dimensions.xacro (robot description, xacro)
@@ -2,7 +2,9 @@
 <robot xmlns:xacro="http://www.ros.org/wiki/xacro">
   <!-- ============ Real hardware dimensions (gobilda parts) ============ -->
-  <!-- gobilda 3601-0014-0120 wheel -->
-  <xacro:property name="wheel_radius" value="0.060"/>
-  <xacro:property name="wheel_width"  value="0.032"/>
+  <!-- gobilda 144mm wheel (meshes/step/wheel_144.step). The previous
+       120mm wheel's files are kept in meshes/ in case we switch back:
+       wheel_120 was radius 0.060, width 0.032. -->
+  <xacro:property name="wheel_radius" value="0.072"/>
+  <xacro:property name="wheel_width"  value="0.052"/>
   <!-- gobilda 1120-series U-channel: every frame part below shares this
        48x48mm cross-section, only the length differs. -->

File: from_pi/src/jessica_description/description/pan_tilt.xacro (robot description, xacro)
@@ -56,5 +56,5 @@
     <origin xyz="0 0 ${servo_height}" rpy="0 0 0"/>
     <axis xyz="0 0 1"/>
-    <limit lower="-1.57" upper="1.57" effort="5.0" velocity="3.0"/>
+    <limit lower="-2.356" upper="2.356" effort="5.0" velocity="3.0"/>
   </joint>
   <link name="tilt_mount">

File: from_pi/src/jessica_description/description/ros2_control.xacro (robot description, xacro)
@@ -10,5 +10,5 @@
       <param name="baud_rate">115200</param>
       <param name="timeout_ms">25</param>   <!-- MUST be < loop period (33ms@30Hz). ReadLine blocks the RT loop up to this long when the ESP32 doesn't reply. -->
-      <param name="wheel_radius">6.0</param>        <!-- cm, used by hardware protocol (gobilda 3601-0014-0120; scales wheel speed + encoder odom) -->
+      <param name="wheel_radius">7.2</param>        <!-- cm, used by hardware protocol (gobilda 144mm wheel; scales wheel speed + encoder odom) -->
       <param name="enc_counts_per_rev">1425</param>
     </hardware>
@@ -50,8 +50,9 @@
     </hardware>
     <!-- Pan-tilt servos: position command + position state.
-         Firmware clamps to its own limits (pan full range, tilt 220-780 units
-         = ±1.32 rad) on top of these. -->
+         Firmware (temp/micropython_servo_control/config.py) clamps to its
+         own limits on top of these: pan 0-1000 units = ±2.356 rad (full
+         servo range), tilt 220-780 units = ±1.32 rad. -->
     <joint name="pan_joint">
-      <command_interface name="position"><param name="min">-1.57</param><param name="max">1.57</param></command_interface>
+      <command_interface name="position"><param name="min">-2.356</param><param name="max">2.356</param></command_interface>
       <state_interface name="position"/>
     </joint>

File: from_pi/src/jessica_description/description/wheels.xacro (robot description, xacro)
@@ -1,11 +1,12 @@
 <?xml version="1.0"?>
 <!--
-  gobilda 3601-0014-0120 wheel (see meshes/step, meshes/visual). Collision
-  stays a plain cylinder primitive rather than the full tread mesh.
-  The mesh's native rotation axis is the STL's local Z; wheel_joint spins
-  about Y, so the visual is rotated -90 deg about X to line the two up, then
-  shifted 16mm (half the wheel width) so the mesh - whose native origin sits
-  at one face, not the centre - ends up centred on the joint like the
-  collision cylinder already is.
+  gobilda 144mm wheel (see meshes/step, meshes/visual; the older wheel_120
+  files are kept there too in case we switch back). Collision stays a plain
+  cylinder primitive rather than the full tread mesh.
+  Unlike wheel_120 (native axis Z, origin at one face), wheel_144's native
+  rotation axis is the STL's local X, spanning -18mm to +34mm - the origin
+  is 8mm off the width's centre. wheel_joint spins about Y, so the visual is
+  yawed +90 deg about Z (native X -> global Y), then shifted -8mm in Y so
+  the mesh ends up centred on the joint like the collision cylinder is.
 -->
 <robot xmlns:xacro="http://www.ros.org/wiki/xacro">
@@ -13,6 +14,6 @@
     <link name="${name}">
       <visual>
-        <origin xyz="0 0.016 0" rpy="${-pi/2} 0 0"/>
-        <geometry><mesh filename="package://jessica_description/description/meshes/visual/wheel_120.stl" scale="0.001 0.001 0.001"/></geometry>
+        <origin xyz="0 -0.008 0" rpy="0 0 ${pi/2}"/>
+        <geometry><mesh filename="package://jessica_description/description/meshes/visual/wheel_144.stl" scale="0.001 0.001 0.001"/></geometry>
         <material name="black"/>
       </visual>

File: robot_pc_ws/src/jessica_description/description/dimensions.xacro (robot description, xacro)
@@ -2,5 +2,7 @@
 <robot xmlns:xacro="http://www.ros.org/wiki/xacro">
   <!-- ============ Real hardware dimensions (gobilda parts) ============ -->
-  <!-- gobilda 3601-0014-0120 wheel -->
+  <!-- gobilda 3601-0014-0120 wheel. The 144mm wheel's files are kept in
+       meshes/ in case we switch again: wheel_144 is radius 0.072, width
+       0.052 (and has a different native axis - see wheels.xacro history). -->
   <xacro:property name="wheel_radius" value="0.060"/>
   <xacro:property name="wheel_width"  value="0.032"/>
@@ -21,5 +23,5 @@
        flag any of these that don't match the real build). -->
   <xacro:property name="wheel_end_inset" value="0.024"/>  <!-- wheel axle inset from each end of a foot -->
-  <xacro:property name="wheel_side_gap"  value="0.020"/>  <!-- gap from the foot's outer face to the wheel's near edge -->
+  <xacro:property name="wheel_side_gap"  value="0.005"/>  <!-- gap from the foot's outer face to the wheel's near edge -->
   <xacro:property name="leg_from_back"   value="0.072"/>  <!-- leg centerline, measured from the back of the foot -->
   <xacro:property name="cross_bar_from_front" value="0.144"/>  <!-- cross-bar centerline, measured from the front of the feet -->

File: robot_pc_ws/src/jessica_description/description/ros2_control.xacro (robot description, xacro)
@@ -1,4 +1,7 @@
 <?xml version="1.0"?>
 <robot xmlns:xacro="http://www.ros.org/wiki/xacro">
+  <!-- Motor controller: ESP32-S3 (USB 303a:1001 → /dev/esp32_motor), 4 wheel
+       motors with encoders. The pan/tilt head moved to its own controller
+       below when the hobby servos were replaced with hiwonder bus servos. -->
   <ros2_control name="JessicaESP32" type="system">
     <hardware>
@@ -7,5 +10,5 @@
       <param name="baud_rate">115200</param>
       <param name="timeout_ms">25</param>   <!-- MUST be < loop period (33ms@30Hz). ReadLine blocks the RT loop up to this long when the ESP32 doesn't reply. -->
-      <param name="wheel_radius">7.2</param>        <!-- cm, used by hardware protocol -->
+      <param name="wheel_radius">6.0</param>        <!-- cm, used by hardware protocol (gobilda 3601-0014-0120; scales wheel speed + encoder odom) -->
       <param name="enc_counts_per_rev">1425</param>
     </hardware>
@@ -31,11 +34,29 @@
       <state_interface name="velocity"/>
     </joint>
-    <!-- Pan-tilt servos: position command + position state (order matters: 4-5) -->
+  </ros2_control>
+  <!-- Head: ESP32 dev board (CH340, USB 1a86:7523 → /dev/esp32_servo) running
+       temp/micropython_servo_control, driving hiwonder bus servos.
+       NOTE: the board reboots when the port opens and homes both servos to
+       centre; the interface waits boot_wait_ms before talking to it. -->
+  <ros2_control name="JessicaServoHead" type="system">
+    <hardware>
+      <plugin>esp32_servo_hardware/ESP32ServoHardware</plugin>
+      <param name="device">/dev/esp32_servo</param>
+      <param name="baud_rate">115200</param>
+      <param name="move_ms">100</param>          <!-- per-command servo move time; short = tracks the trajectory stream closely -->
+      <param name="boot_wait_ms">3000</param>
+      <param name="state_refresh_ms">1000</param>   <!-- idle "pos" poll period -->
+      <param name="min_send_period_ms">100</param>  <!-- floor between ptr sends; faster overflows the board's UART -->
+    </hardware>
+    <!-- Pan-tilt servos: position command + position state.
+         Firmware (temp/micropython_servo_control/config.py) clamps to its
+         own limits on top of these: pan 0-1000 units = ±2.356 rad (full
+         servo range), tilt 220-780 units = ±1.32 rad. -->
     <joint name="pan_joint">
-      <command_interface name="position"><param name="min">-1.57</param><param name="max">1.57</param></command_interface>
+      <command_interface name="position"><param name="min">-2.356</param><param name="max">2.356</param></command_interface>
       <state_interface name="position"/>
     </joint>
     <joint name="tilt_joint">
-      <command_interface name="position"><param name="min">-1.5</param><param name="max">0.87</param></command_interface>
+      <command_interface name="position"><param name="min">-1.3</param><param name="max">0.87</param></command_interface>
       <state_interface name="position"/>
     </joint>

File: robot_pc_ws/src/jessica_description/description/wheels.xacro (robot description, xacro)
@@ -1,5 +1,6 @@
 <?xml version="1.0"?>
 <!--
-  gobilda 3601-0014-0120 wheel (see meshes/step, meshes/visual). Collision
+  gobilda 3601-0014-0120 wheel (see meshes/step, meshes/visual; the
+  wheel_144 files are kept there too in case we switch again). Collision
   stays a plain cylinder primitive rather than the full tread mesh.
   The mesh's native rotation axis is the STL's local Z; wheel_joint spins
@@ -7,5 +8,6 @@
   shifted 16mm (half the wheel width) so the mesh - whose native origin sits
   at one face, not the centre - ends up centred on the joint like the
-  collision cylinder already is.
+  collision cylinder already is. (wheel_144 is different: native axis X,
+  origin 8mm off-centre -> xyz="0 -0.008 0" rpy="0 0 pi/2" if reinstated.)
 -->
 <robot xmlns:xacro="http://www.ros.org/wiki/xacro">

Commit message: pi stuff updated

File: from_pi/src/jessica_description/description/dimensions.xacro (robot description, xacro)
@@ -2,9 +2,9 @@
 <robot xmlns:xacro="http://www.ros.org/wiki/xacro">
   <!-- ============ Real hardware dimensions (gobilda parts) ============ -->
-  <!-- gobilda 144mm wheel (meshes/step/wheel_144.step). The previous
-       120mm wheel's files are kept in meshes/ in case we switch back:
-       wheel_120 was radius 0.060, width 0.032. -->
-  <xacro:property name="wheel_radius" value="0.072"/>
-  <xacro:property name="wheel_width"  value="0.052"/>
+  <!-- gobilda 3601-0014-0120 wheel. The 144mm wheel's files are kept in
+       meshes/ in case we switch again: wheel_144 is radius 0.072, width
+       0.052 (and has a different native axis - see wheels.xacro history). -->
+  <xacro:property name="wheel_radius" value="0.060"/>
+  <xacro:property name="wheel_width"  value="0.032"/>
   <!-- gobilda 1120-series U-channel: every frame part below shares this
        48x48mm cross-section, only the length differs. -->

File: from_pi/src/jessica_description/description/ros2_control.xacro (robot description, xacro)
@@ -10,5 +10,5 @@
       <param name="baud_rate">115200</param>
       <param name="timeout_ms">25</param>   <!-- MUST be < loop period (33ms@30Hz). ReadLine blocks the RT loop up to this long when the ESP32 doesn't reply. -->
-      <param name="wheel_radius">7.2</param>        <!-- cm, used by hardware protocol (gobilda 144mm wheel; scales wheel speed + encoder odom) -->
+      <param name="wheel_radius">6.0</param>        <!-- cm, used by hardware protocol (gobilda 3601-0014-0120; scales wheel speed + encoder odom) -->
       <param name="enc_counts_per_rev">1425</param>
     </hardware>

File: from_pi/src/jessica_description/description/wheels.xacro (robot description, xacro)
@@ -1,12 +1,13 @@
 <?xml version="1.0"?>
 <!--
-  gobilda 144mm wheel (see meshes/step, meshes/visual; the older wheel_120
-  files are kept there too in case we switch back). Collision stays a plain
-  cylinder primitive rather than the full tread mesh.
-  Unlike wheel_120 (native axis Z, origin at one face), wheel_144's native
-  rotation axis is the STL's local X, spanning -18mm to +34mm - the origin
-  is 8mm off the width's centre. wheel_joint spins about Y, so the visual is
-  yawed +90 deg about Z (native X -> global Y), then shifted -8mm in Y so
-  the mesh ends up centred on the joint like the collision cylinder is.
+  gobilda 3601-0014-0120 wheel (see meshes/step, meshes/visual; the
+  wheel_144 files are kept there too in case we switch again). Collision
+  stays a plain cylinder primitive rather than the full tread mesh.
+  The mesh's native rotation axis is the STL's local Z; wheel_joint spins
+  about Y, so the visual is rotated -90 deg about X to line the two up, then
+  shifted 16mm (half the wheel width) so the mesh - whose native origin sits
+  at one face, not the centre - ends up centred on the joint like the
+  collision cylinder already is. (wheel_144 is different: native axis X,
+  origin 8mm off-centre -> xyz="0 -0.008 0" rpy="0 0 pi/2" if reinstated.)
 -->
 <robot xmlns:xacro="http://www.ros.org/wiki/xacro">
@@ -14,6 +15,6 @@
     <link name="${name}">
       <visual>
-        <origin xyz="0 -0.008 0" rpy="0 0 ${pi/2}"/>
-        <geometry><mesh filename="package://jessica_description/description/meshes/visual/wheel_144.stl" scale="0.001 0.001 0.001"/></geometry>
+        <origin xyz="0 0.016 0" rpy="${-pi/2} 0 0"/>
+        <geometry><mesh filename="package://jessica_description/description/meshes/visual/wheel_120.stl" scale="0.001 0.001 0.001"/></geometry>
         <material name="black"/>
       </visual>
